File: PCB/auto-chicken-coop-door.sch (KiCad schematic (older format))
At the start: 15 parts, among them J1 Programming_Headers, M1 Motor_DC, SW1 SW_Right, SW2 SW_Middle, SW3 SW_Left, U1 Arduino_Pro_Mini, U2 DS3231M, U3 Sparkfun_Dual_Motor_Driver_TB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, U4 OLED_Display_128x68, U5 Adafruit_Solar_Charger_390

Commit message: Change buttons to connectors
Parts:
- removed SW1: SW_Right, symbol Switch:SW_Push_Dual
- removed SW2: SW_Middle, symbol Switch:SW_Push_Dual
- removed SW3: SW_Left, symbol Switch:SW_Push_Dual
- added J2: Pushbutton_Left, symbol Connector_Generic:Conn_01x02
- added J3: Pushbutton_Middle, symbol Connector_Generic:Conn_01x02
- added J4: Pushbutton_Right, symbol Connector_Generic:Conn_01x02
Connections:
- wire segments 64 -> 58
Other:
- moved on the sheet: BT1, J1, M1, R1, SC1, U2

Commit message: Add pushbuttons; add motor input voltage to 7.5V
Parts:
- added J5: Conn_Left, symbol Connector_Generic:Conn_01x02
- added J6: Conn_Middle, symbol Connector_Generic:Conn_01x02
- added J7: Conn_Right, symbol Connector_Generic:Conn_01x02
- added SW1: SW_Left, symbol Switch:SW_Push
- added SW2: SW_Middle, symbol Switch:SW_Push
- added SW3: SW_Right, symbol Switch:SW_Push
- J2: value Pushbutton_Left -> Conn_Left
- J3: value Pushbutton_Middle -> Conn_Middle
- J4: value Pushbutton_Right -> Conn_Right
Connections:
- net labels added: +7.5V
- wire segments 58 -> 78
Other:
- moved on the sheet: BT1, J1, J2, J3, J4, M1, R1, R2, R3, SC1, U2
