File: PCB/auto-chicken-coop-door.sch (KiCad schematic (older format))
At the start: 21 parts, among them J1 Programming_Headers, J2 Conn_Left, J3 Conn_Middle, J4 Conn_Right, J5 Conn_Left, J6 Conn_Middle, J7 Conn_Right, M1 Motor_DC, SW1 SW_Left, SW2 SW_Middle, SW3 SW_Right, U1 Arduino_Pro_Mini, U2 DS3231M, U3 Sparkfun_Dual_Motor_Driver_TB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, U4 OLED_Display_128x68, U5 Adafruit_Solar_Charger_390

Commit message: Add TIP122 and buck/boost module to schematic
Parts:
- added Q1: TIP122, Package_TO_SOT_THT:TO-220-3_Vertical, symbol Transistor_BJT:TIP122
- added U6: Buck_Boost_XL6009E1, symbol Chicken~Coop~Door:Buck_Boost_module
Connections:
- net labels removed: +7.5V
- wire segments 78 -> 98
Other:
- moved on the sheet: U2
Changed lines of the file:
@@
 EESchema Schematic File Version 4
+LIBS:auto-chicken-coop-door-cache
 EELAYER 29 0
 EELAYER END
@@
 $EndDescr
 $Comp
-L Timer_RTC:DS3231M U2
-U 1 1 5CC70780
-P 2800 2750
-F 0 "U2" H 3300 2450 50  0000 C CNN
-F 1 "DS3231M" H 3150 2350 50  0000 C CNN
-F 2 "Package_SO:SOIC-16W_7.5x10.3mm_P1.27mm" H 2800 2150 50  0001 C CNN
-F 3 "http://datasheets.maximintegrated.com/en/ds/DS3231.pdf" H 3070 2800 50  0001 C CNN
-	1    2800 2750
-	1    0    0    -1
-$EndComp
-$Comp
 L Chicken~Coop~Door:OLED_Display_128x68 U4
 U 1 1 5CC7AC9B
@@
 $EndComp
 Wire Wire Line
-	3300 2850 4150 2850
-Wire Wire Line
-	4150 2850 4150 3750
-Wire Wire Line
-	4150 3750 4900 3750
-Wire Wire Line
 	4100 4750 4100 4450
 Wire Wire Line
@@
 L power:VCC #PWR0102
 U 1 1 5CD03543
-P 1950 4750
-F 0 "#PWR0102" H 1950 4600 50  0001 C CNN
-F 1 "VCC" H 1967 4923 50  0000 C CNN
-F 2 "" H 1950 4750 50  0001 C CNN
-F 3 "" H 1950 4750 50  0001 C CNN
-	1    1950 4750
+P 2100 4750
+F 0 "#PWR0102" H 2100 4600 50  0001 C CNN
+F 1 "VCC" H 2117 4923 50  0000 C CNN
+F 2 "" H 2100 4750 50  0001 C CNN
+F 3 "" H 2100 4750 50  0001 C CNN
+	1    2100 4750
 	1    0    0    -1
 $EndComp
@@
 Text GLabel 5500 5300 2    50   Input ~ 0
 SCL
-Text GLabel 2300 2650 0    50   Input ~ 0
+Text GLabel 3300 3300 0    50   Input ~ 0
 SDA
-Text GLabel 2300 2550 0    50   Input ~ 0
+Text GLabel 3300 3200 0    50   Input ~ 0
 SCL
 $Comp
 L power:VCC #PWR0103
 U 1 1 5CD79418
-P 2700 2350
-F 0 "#PWR0103" H 2700 2200 50  0001 C CNN
-F 1 "VCC" H 2717 2523 50  0000 C CNN
-F 2 "" H 2700 2350 50  0001 C CNN
-F 3 "" H 2700 2350 50  0001 C CNN
-	1    2700 2350
+P 3700 3000
+F 0 "#PWR0103" H 3700 2850 50  0001 C CNN
+F 1 "VCC" H 3717 3173 50  0000 C CNN
+F 2 "" H 3700 3000 50  0001 C CNN
+F 3 "" H 3700 3000 50  0001 C CNN
+	1    3700 3000
 	1    0    0    -1
 $EndComp
@@
 L power:GND #PWR0104
 U 1 1 5CD7EE85
-P 2800 3150
-F 0 "#PWR0104" H 2800 2900 50  0001 C CNN
-F 1 "GND" H 2805 2977 50  0000 C CNN
-F 2 "" H 2800 3150 50  0001 C CNN
-F 3 "" H 2800 3150 50  0001 C CNN
-	1    2800 3150
+P 3800 3800
+F 0 "#PWR0104" H 3800 3550 50  0001 C CNN
+F 1 "GND" H 3805 3627 50  0000 C CNN
+F 2 "" H 3800 3800 50  0001 C CNN
+F 3 "" H 3800 3800 50  0001 C CNN
+	1    3800 3800
 	1    0    0    -1
 $EndComp
@@
 	6300 3300 7200 3300
 Wire Wire Line
-	7200 2000 7200 3300
-Wire Wire Line
-	7300 2000 7300 3400
+	7200 2000 7200 2550
+Wire Wire Line
+	7300 2000 7300 2450
 Connection ~ 7300 3400
 $Comp
@@
 Wire Wire Line
 	10050 5450 9900 5450
-$Comp
-L power:+7.5V #PWR0115
-U 1 1 5CF3B40F
-P 2200 4750
-F 0 "#PWR0115" H 2200 4600 50  0001 C CNN
-F 1 "+7.5V" H 2215 4923 50  0000 C CNN
-F 2 "" H 2200 4750 50  0001 C CNN
-F 3 "" H 2200 4750 50  0001 C CNN
-	1    2200 4750
-	1    0    0    -1
-$EndComp
-Wire Wire Line
-	2200 4750 2350 4750
-Wire Wire Line
-	1950 4750 1950 4850
-Wire Wire Line
-	1950 4850 2350 4850
+Wire Wire Line
+	2100 4750 2100 4850
+$Comp
+L Timer_RTC:DS3231M U2
+U 1 1 5CC70780
+P 3800 3400
+F 0 "U2" H 4300 3100 50  0000 C CNN
+F 1 "DS3231M" H 4150 3000 50  0000 C CNN
+F 2 "Package_SO:SOIC-16W_7.5x10.3mm_P1.27mm" H 3800 2800 50  0001 C CNN
+F 3 "http://datasheets.maximintegrated.com/en/ds/DS3231.pdf" H 4070 3450 50  0001 C CNN
+	1    3800 3400
+	1    0    0    -1
+$EndComp
+Wire Wire Line
+	4650 3500 4300 3500
+$Comp
+L Chicken~Coop~Door:Buck_Boost_module U6
+U 1 1 5CEF5879
+P 3750 2150
+F 0 "U6" H 3750 1885 50  0000 C CNN
+F 1 "Buck_Boost_XL6009E1" H 3750 1976 50  0000 C CNN
+F 2 "" H 3900 2100 50  0001 C CNN
+F 3 "" H 3900 2100 50  0001 C CNN
+	1    3750 2150
+	-1   0    0    1
+$EndComp
+Wire Wire Line
+	5550 2250 5550 2550
+Wire Wire Line
+	5550 2550 7200 2550
+Connection ~ 7200 2550
+Wire Wire Line
+	7200 2550 7200 3300
+Wire Wire Line
+	4100 2100 5650 2100
+Wire Wire Line
+	5650 2100 5650 2450
+Wire Wire Line
+	5650 2450 7300 2450
+Connection ~ 7300 2450
+Wire Wire Line
+	7300 2450 7300 3400
+Wire Wire Line
+	3400 2250 2250 2250
+Wire Wire Line
+	2250 2250 2250 4750
+Wire Wire Line
+	2250 4750 2350 4750
+Wire Wire Line
+	1950 4950 2350 4950
+Wire Wire Line
+	3400 2100 1950 2100
+Wire Wire Line
+	1950 2100 1950 4950
+Wire Wire Line
+	2100 4850 2350 4850
+$Comp
+L Transistor_BJT:TIP122 Q1
+U 1 1 5CF1402B
+P 4750 2450
+F 0 "Q1" H 5050 2450 50  0000 C CNN
+F 1 "TIP122" H 5050 2350 50  0000 C CNN
+F 2 "Package_TO_SOT_THT:TO-220-3_Vertical" H 4950 2375 50  0001 L CIN
+F 3 "http://www.fairchildsemi.com/ds/TI/TIP120.pdf" H 4750 2450 50  0001 L CNN
+	1    4750 2450
+	1    0    0    -1
+$EndComp
+Wire Wire Line
+	4100 2250 4150 2250
+Wire Wire Line
+	4750 3750 4900 3750
+Wire Wire Line
+	4650 3850 4900 3850
+Wire Wire Line
+	4650 3500 4650 3850
+Wire Wire Line
+	4550 2450 4550 3250
+Wire Wire Line
+	4550 3250 4750 3250
+Wire Wire Line
+	4750 3250 4750 3750
+Wire Wire Line
+	4150 2650 4850 2650
+Wire Wire Line
+	4150 2250 4150 2650
+Wire Wire Line
+	4850 2250 5550 2250
 $EndSCHEMATC
