File: PCB/auto-chicken-coop-door.sch (KiCad schematic (older format))
At the start: 23 parts, among them J1 Programming_Headers, J2 Conn_Left, J3 Conn_Middle, J4 Conn_Right, J5 Conn_Left, J6 Conn_Middle, J7 Conn_Right, M1 Motor_DC, Q1 TIP122, SW1 SW_Left, SW2 SW_Middle, SW3 SW_Right, U1 Arduino_Pro_Mini, U2 DS3231M, U3 Sparkfun_Dual_Motor_Driver_TB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, U4 OLED_Display_128x68, U5 Adafruit_Solar_Charger_390, U6 Buck_Boost_XL6009E1

Commit message: Update schematic with pins and correct transistor config
Use TIP122 to enable/disable the XL6009 module. Doesn't work if enable is connected
directly to pin 10.
Parts:
- added R4: 1k, symbol Device:R
Connections:
- net labels added: D10, D3, D4, D5
- wire segments 98 -> 88
Other:
- moved on the sheet: Q1, U2
Changed lines of the file:
@@
 Text GLabel 5500 5300 2    50   Input ~ 0
 SCL
-Text GLabel 3300 3300 0    50   Input ~ 0
+Text GLabel 2700 3550 0    50   Input ~ 0
 SDA
-Text GLabel 3300 3200 0    50   Input ~ 0
+Text GLabel 2700 3450 0    50   Input ~ 0
 SCL
 $Comp
 L power:VCC #PWR0103
 U 1 1 5CD79418
-P 3700 3000
-F 0 "#PWR0103" H 3700 2850 50  0001 C CNN
-F 1 "VCC" H 3717 3173 50  0000 C CNN
-F 2 "" H 3700 3000 50  0001 C CNN
-F 3 "" H 3700 3000 50  0001 C CNN
-	1    3700 3000
+P 3100 3250
+F 0 "#PWR0103" H 3100 3100 50  0001 C CNN
+F 1 "VCC" H 3117 3423 50  0000 C CNN
+F 2 "" H 3100 3250 50  0001 C CNN
+F 3 "" H 3100 3250 50  0001 C CNN
+	1    3100 3250
 	1    0    0    -1
 $EndComp
@@
 L power:GND #PWR0104
 U 1 1 5CD7EE85
-P 3800 3800
-F 0 "#PWR0104" H 3800 3550 50  0001 C CNN
-F 1 "GND" H 3805 3627 50  0000 C CNN
-F 2 "" H 3800 3800 50  0001 C CNN
-F 3 "" H 3800 3800 50  0001 C CNN
-	1    3800 3800
+P 3200 4050
+F 0 "#PWR0104" H 3200 3800 50  0001 C CNN
+F 1 "GND" H 3205 3877 50  0000 C CNN
+F 2 "" H 3200 4050 50  0001 C CNN
+F 3 "" H 3200 4050 50  0001 C CNN
+	1    3200 4050
 	1    0    0    -1
 $EndComp
@@
 	1    0    0    -1
 $EndComp
-Wire Wire Line
-	6300 4350 7600 4350
-Wire Wire Line
-	7600 4350 7600 3400
-Connection ~ 8250 3400
 $Comp
 L power:VCC #PWR0111
@@
 	1    0    0    -1
 $EndComp
-Connection ~ 8250 4450
-Wire Wire Line
-	6300 4550 7600 4550
-Wire Wire Line
-	7600 4550 7600 5350
-Connection ~ 8250 5350
 $Comp
 L Connector_Generic:Conn_01x02 J5
@@
 Wire Wire Line
 	10050 3500 9900 3500
-Wire Wire Line
-	6300 4450 8250 4450
-Wire Wire Line
-	7600 3400 8250 3400
-Wire Wire Line
-	7600 5350 8250 5350
 $Comp
 L Connector_Generic:Conn_01x02 J6
@@
 L Timer_RTC:DS3231M U2
 U 1 1 5CC70780
-P 3800 3400
-F 0 "U2" H 4300 3100 50  0000 C CNN
-F 1 "DS3231M" H 4150 3000 50  0000 C CNN
-F 2 "Package_SO:SOIC-16W_7.5x10.3mm_P1.27mm" H 3800 2800 50  0001 C CNN
-F 3 "http://datasheets.maximintegrated.com/en/ds/DS3231.pdf" H 4070 3450 50  0001 C CNN
-	1    3800 3400
-	1    0    0    -1
-$EndComp
-Wire Wire Line
-	4650 3500 4300 3500
+P 3200 3650
+F 0 "U2" H 3700 3350 50  0000 C CNN
+F 1 "DS3231M" H 3550 3250 50  0000 C CNN
+F 2 "Package_SO:SOIC-16W_7.5x10.3mm_P1.27mm" H 3200 3050 50  0001 C CNN
+F 3 "http://datasheets.maximintegrated.com/en/ds/DS3231.pdf" H 3470 3700 50  0001 C CNN
+	1    3200 3650
+	1    0    0    -1
+$EndComp
 $Comp
 L Chicken~Coop~Door:Buck_Boost_module U6
 U 1 1 5CEF5879
-P 3750 2150
-F 0 "U6" H 3750 1885 50  0000 C CNN
-F 1 "Buck_Boost_XL6009E1" H 3750 1976 50  0000 C CNN
-F 2 "" H 3900 2100 50  0001 C CNN
-F 3 "" H 3900 2100 50  0001 C CNN
-	1    3750 2150
+P 3750 1700
+F 0 "U6" H 3750 1435 50  0000 C CNN
+F 1 "Buck_Boost_XL6009E1" H 3750 1526 50  0000 C CNN
+F 2 "" H 3900 1650 50  0001 C CNN
+F 3 "" H 3900 1650 50  0001 C CNN
+	1    3750 1700
 	-1   0    0    1
 $EndComp
-Wire Wire Line
-	5550 2250 5550 2550
 Wire Wire Line
 	5550 2550 7200 2550
@@
 	7200 2550 7200 3300
 Wire Wire Line
-	4100 2100 5650 2100
-Wire Wire Line
-	5650 2100 5650 2450
-Wire Wire Line
 	5650 2450 7300 2450
 Connection ~ 7300 2450
@@
 	7300 2450 7300 3400
 Wire Wire Line
-	3400 2250 2250 2250
-Wire Wire Line
-	2250 2250 2250 4750
-Wire Wire Line
 	2250 4750 2350 4750
 Wire Wire Line
 	1950 4950 2350 4950
-Wire Wire Line
-	3400 2100 1950 2100
-Wire Wire Line
-	1950 2100 1950 4950
 Wire Wire Line
 	2100 4850 2350 4850
@@
 L Transistor_BJT:TIP122 Q1
 U 1 1 5CF1402B
-P 4750 2450
-F 0 "Q1" H 5050 2450 50  0000 C CNN
-F 1 "TIP122" H 5050 2350 50  0000 C CNN
-F 2 "Package_TO_SOT_THT:TO-220-3_Vertical" H 4950 2375 50  0001 L CIN
-F 3 "http://www.fairchildsemi.com/ds/TI/TIP120.pdf" H 4750 2450 50  0001 L CNN
-	1    4750 2450
-	1    0    0    -1
-$EndComp
-Wire Wire Line
-	4100 2250 4150 2250
-Wire Wire Line
-	4550 2450 4550 3250
-Wire Wire Line
-	4550 3250 4750 3250
-Wire Wire Line
-	4150 2650 4850 2650
-Wire Wire Line
-	4150 2250 4150 2650
-Wire Wire Line
-	4850 2250 5550 2250
-Wire Wire Line
-	4650 3500 4650 3750
-Wire Wire Line
-	4650 3750 4900 3750
-Wire Wire Line
-	4750 3250 4750 3850
-Wire Wire Line
-	4750 3850 4900 3850
+P 3650 2300
+F 0 "Q1" H 3950 2300 50  0000 C CNN
+F 1 "TIP122" H 3950 2200 50  0000 C CNN
+F 2 "Package_TO_SOT_THT:TO-220-3_Vertical" H 3850 2225 50  0001 L CIN
+F 3 "http://www.fairchildsemi.com/ds/TI/TIP120.pdf" H 3650 2300 50  0001 L CNN
+	1    3650 2300
+	1    0    0    -1
+$EndComp
+$Comp
+L Device:R R4
+U 1 1 5CF6B441
+P 3250 2300
+F 0 "R4" V 3150 2250 50  0000 L CNN
+F 1 "1k" V 3320 2255 50  0000 L CNN
+F 2 "" V 3180 2300 50  0001 C CNN
+F 3 "~" H 3250 2300 50  0001 C CNN
+	1    3250 2300
+	0    1    1    0
+$EndComp
+Wire Wire Line
+	4150 1800 5550 1800
+Wire Wire Line
+	4150 1650 5650 1650
+$Comp
+L power:GND #PWR?
+U 1 1 5CF9556B
+P 3750 2500
+F 0 "#PWR?" H 3750 2250 50  0001 C CNN
+F 1 "GND" H 3755 2327 50  0000 C CNN
+F 2 "" H 3750 2500 50  0001 C CNN
+F 3 "" H 3750 2500 50  0001 C CNN
+	1    3750 2500
+	1    0    0    -1
+$EndComp
+Text GLabel 2950 2300 0    50   Input ~ 0
+D10
+Wire Wire Line
+	2950 2300 3100 2300
+Wire Wire Line
+	3400 2300 3450 2300
+Text GLabel 6300 4550 2    50   Input ~ 0
+D10
+Wire Wire Line
+	3700 3750 4900 3750
+Wire Wire Line
+	3750 2100 3750 1950
+Wire Wire Line
+	2250 1800 2250 4750
+Wire Wire Line
+	1950 1650 1950 4950
+Wire Wire Line
+	5550 1800 5550 2550
+Wire Wire Line
+	5650 1650 5650 2450
+Wire Wire Line
+	1950 1650 3300 1650
+Wire Wire Line
+	3300 1800 2250 1800
+Wire Wire Line
+	8050 4450 8250 4450
+Connection ~ 8250 4450
+Text GLabel 8050 4450 0    50   Input ~ 0
+D3
+Text GLabel 4900 3850 0    50   Input ~ 0
+D3
+Text GLabel 4900 3950 0    50   Input ~ 0
+D4
+Text GLabel 4900 4050 0    50   Input ~ 0
+D5
+Text GLabel 8050 5350 0    50   Input ~ 0
+D4
+Text GLabel 8050 3400 0    50   Input ~ 0
+D5
+Wire Wire Line
+	8050 5350 8250 5350
+Connection ~ 8250 5350
+Wire Wire Line
+	8050 3400 8250 3400
+Connection ~ 8250 3400
 $EndSCHEMATC

Commit message: Add footprints to schematic
Parts:
- removed U2: DS3231M, Package_SO:SOIC-16W_7.5x10.3mm_P1.27mm, symbol Timer_RTC:DS3231M
- removed U4: OLED_Display_128x68, symbol Chicken~Coop~Door:OLED_Display_128x68
- added J10, J11: Charger, Connector_JST:JST_XH_B02B-XH-A_1x02_P2.50mm_Vertical, symbol Connector_Generic:Conn_01x02
- added J8: Conn_01x01, TestPoint:TestPoint_THTPad_D2.0mm_Drill1.0mm, symbol Connector_Generic:Conn_01x01
- added J9: BuckBoost, Connector_JST:JST_XH_B02B-XH-A_1x02_P2.50mm_Vertical, symbol Connector_Generic:Conn_01x02
- added U2: DS3231, Connector_PinSocket_2.54mm:PinSocket_1x06_P2.54mm_Vertical, symbol sensors:DS3231
- added U4: SSD1306_OLED_128x32, personal:SSD1306_Adafruit_128x32, symbol sensors:SSD1306_OLED_128x32
- J2, J3, J4, M1: footprint (none) -> Connector_JST:JST_XH_B02B-XH-A_1x02_P2.50mm_Vertical
- R1, R2, R3, R4: footprint (none) -> Resistor_THT:R_Axial_DIN0204_L3.6mm_D1.6mm_P7.62mm_Horizontal
- U1: footprint (none) -> personal:ArduinoProMini
- U3: footprint (none) -> personal:Sparkfun_TB6612FNG
Connections:
- wire segments 88 -> 105
Changed lines of the file:
@@
 EESchema Schematic File Version 4
 LIBS:auto-chicken-coop-door-cache
-EELAYER 29 0
+EELAYER 26 0
 EELAYER END
 $Descr A4 11693 8268
@@
 Comment4 ""
 $EndDescr
-$Comp
-L Chicken~Coop~Door:OLED_Display_128x68 U4
-U 1 1 5CC7AC9B
-P 5050 6100
-F 0 "U4" H 4950 6650 50  0000 C CNN
-F 1 "OLED_Display_128x68" H 5050 6100 50  0000 C CNN
-F 2 "" H 5050 6100 50  0001 C CNN
-F 3 "" H 5050 6100 50  0001 C CNN
-	1    5050 6100
-	1    0    0    -1
-$EndComp
 Wire Wire Line
 	4100 4750 4100 4450
@@
 F 0 "U3" H 2750 5750 50  0000 C CNN
 F 1 "Sparkfun_Dual_Motor_Driver_TB6612FNG" H 2750 5650 50  0000 C CNN
-F 2 "" H 2750 5700 50  0001 C CNN
+F 2 "personal:Sparkfun_TB6612FNG" H 2750 5700 50  0001 C CNN
 F 3 "" H 2750 5700 50  0001 C CNN
 	1    2750 5700
@@
 F 0 "M1" H 1458 5046 50  0000 L CNN
 F 1 "Motor_DC" H 1458 4955 50  0000 L CNN
-F 2 "" H 1300 4960 50  0001 C CNN
+F 2 "Connector_JST:JST_XH_B02B-XH-A_1x02_P2.50mm_Vertical" H 1300 4960 50  0001 C CNN
 F 3 "~" H 1300 4960 50  0001 C CNN
 	1    1300 5050
 	1    0    0    -1
 $EndComp
-Wire Wire Line
-	5400 5650 5300 5650
-Wire Wire Line
-	5500 4750 5500 5750
-Wire Wire Line
-	5500 5750 5300 5750
 Text GLabel 5400 5150 0    50   Input ~ 0
 SDA
 Text GLabel 5500 5300 2    50   Input ~ 0
 SCL
-Text GLabel 2700 3550 0    50   Input ~ 0
+Text GLabel 3000 3500 0    50   Input ~ 0
 SDA
-Text GLabel 2700 3450 0    50   Input ~ 0
+Text GLabel 3000 3400 0    50   Input ~ 0
 SCL
 $Comp
 L power:VCC #PWR0103
 U 1 1 5CD79418
-P 3100 3250
-F 0 "#PWR0103" H 3100 3100 50  0001 C CNN
-F 1 "VCC" H 3117 3423 50  0000 C CNN
-F 2 "" H 3100 3250 50  0001 C CNN
-F 3 "" H 3100 3250 50  0001 C CNN
-	1    3100 3250
+P 3700 3200
+F 0 "#PWR0103" H 3700 3050 50  0001 C CNN
+F 1 "VCC" H 3717 3373 50  0000 C CNN
+F 2 "" H 3700 3200 50  0001 C CNN
+F 3 "" H 3700 3200 50  0001 C CNN
+	1    3700 3200
 	1    0    0    -1
 $EndComp
@@
 L power:GND #PWR0104
 U 1 1 5CD7EE85
-P 3200 4050
-F 0 "#PWR0104" H 3200 3800 50  0001 C CNN
-F 1 "GND" H 3205 3877 50  0000 C CNN
-F 2 "" H 3200 4050 50  0001 C CNN
-F 3 "" H 3200 4050 50  0001 C CNN
-	1    3200 4050
-	1    0    0    -1
-$EndComp
-Wire Wire Line
-	5400 4750 5400 5650
+P 3700 3500
+F 0 "#PWR0104" H 3700 3250 50  0001 C CNN
+F 1 "GND" H 3705 3327 50  0000 C CNN
+F 2 "" H 3700 3500 50  0001 C CNN
+F 3 "" H 3700 3500 50  0001 C CNN
+	1    3700 3500
+	1    0    0    -1
+$EndComp
 $Comp
 L power:VCC #PWR0105
 U 1 1 5CDDF751
-P 5700 5850
-F 0 "#PWR0105" H 5700 5700 50  0001 C CNN
-F 1 "VCC" H 5717 6023 50  0000 C CNN
-F 2 "" H 5700 5850 50  0001 C CNN
-F 3 "" H 5700 5850 50  0001 C CNN
-	1    5700 5850
+P 5250 5850
+F 0 "#PWR0105" H 5250 5700 50  0001 C CNN
+F 1 "VCC" H 5267 6023 50  0000 C CNN
+F 2 "" H 5250 5850 50  0001 C CNN
+F 3 "" H 5250 5850 50  0001 C CNN
+	1    5250 5850
 	1    0    0    -1
 $EndComp
@@
 L power:GND #PWR0106
 U 1 1 5CDE402A
-P 5700 5950
-F 0 "#PWR0106" H 5700 5700 50  0001 C CNN
-F 1 "GND" H 5705 5777 50  0000 C CNN
-F 2 "" H 5700 5950 50  0001 C CNN
-F 3 "" H 5700 5950 50  0001 C CNN
-	1    5700 5950
-	1    0    0    -1
-$EndComp
-Wire Wire Line
-	5700 5950 5300 5950
-Wire Wire Line
-	5300 5850 5700 5850
+P 5250 5950
+F 0 "#PWR0106" H 5250 5700 50  0001 C CNN
+F 1 "GND" H 5255 5777 50  0000 C CNN
+F 2 "" H 5250 5950 50  0001 C CNN
+F 3 "" H 5250 5950 50  0001 C CNN
+	1    5250 5950
+	1    0    0    -1
+$EndComp
 $Comp
 L Chicken~Coop~Door:Adafruit_Solar_Charger_390 U5
@@
 U 1 1 5CC9C424
 P 5600 3950
-F 0 "U1" H 6100 3150 50  0000 C CNN
-F 1 "Arduino_Pro_Mini" H 6100 3050 50  0000 C CNN
-F 2 "" H 6350 3050 50  0001 C CNN
+F 0 "U1" H 5950 3150 50  0000 C CNN
+F 1 "Arduino_Pro_Mini" H 5900 3000 50  0000 C CNN
+F 2 "personal:ArduinoProMini" H 6350 3050 50  0001 C CNN
 F 3 "" H 6350 3050 50  0001 C CNN
 	1    5600 3950
@@
 F 0 "R1" H 8320 3296 50  0000 L CNN
 F 1 "10k" H 8320 3205 50  0000 L CNN
-F 2 "" V 8180 3250 50  0001 C CNN
+F 2 "Resistor_THT:R_Axial_DIN0204_L3.6mm_D1.6mm_P7.62mm_Horizontal" V 8180 3250 50  0001 C CNN
 F 3 "~" H 8250 3250 50  0001 C CNN
 	1    8250 3250
@@
 F 0 "J2" H 8780 3392 50  0000 L CNN
 F 1 "Conn_Left" H 8780 3301 50  0000 L CNN
-F 2 "" H 8700 3400 50  0001 C CNN
+F 2 "Connector_JST:JST_XH_B02B-XH-A_1x02_P2.50mm_Vertical" H 8700 3400 50  0001 C CNN
 F 3 "~" H 8700 3400 50  0001 C CNN
 	1    8700 3400
@@
 F 0 "R2" H 8320 4346 50  0000 L CNN
 F 1 "10k" H 8320 4255 50  0000 L CNN
-F 2 "" V 8180 4300 50  0001 C CNN
+F 2 "Resistor_THT:R_Axial_DIN0204_L3.6mm_D1.6mm_P7.62mm_Horizontal" V 8180 4300 50  0001 C CNN
 F 3 "~" H 8250 4300 50  0001 C CNN
 	1    8250 4300
@@
 F 0 "J3" H 8780 4442 50  0000 L CNN
 F 1 "Conn_Middle" H 8780 4351 50  0000 L CNN
-F 2 "" H 8700 4450 50  0001 C CNN
+F 2 "Connector_JST:JST_XH_B02B-XH-A_1x02_P2.50mm_Vertical" H 8700 4450 50  0001 C CNN
 F 3 "~" H 8700 4450 50  0001 C CNN
 	1    8700 4450
@@
 F 0 "R3" H 8320 5246 50  0000 L CNN
 F 1 "10k" H 8320 5155 50  0000 L CNN
-F 2 "" V 8180 5200 50  0001 C CNN
+F 2 "Resistor_THT:R_Axial_DIN0204_L3.6mm_D1.6mm_P7.62mm_Horizontal" V 8180 5200 50  0001 C CNN
 F 3 "~" H 8250 5200 50  0001 C CNN
 	1    8250 5200
@@
 F 0 "J4" H 8780 5342 50  0000 L CNN
 F 1 "Conn_Right" H 8780 5251 50  0000 L CNN
-F 2 "" H 8700 5350 50  0001 C CNN
+F 2 "Connector_JST:JST_XH_B02B-XH-A_1x02_P2.50mm_Vertical" H 8700 5350 50  0001 C CNN
 F 3 "~" H 8700 5350 50  0001 C CNN
 	1    8700 5350
@@
 	2100 4750 2100 4850
 $Comp
-L Timer_RTC:DS3231M U2
-U 1 1 5CC70780
-P 3200 3650
-F 0 "U2" H 3700 3350 50  0000 C CNN
-F 1 "DS3231M" H 3550 3250 50  0000 C CNN
-F 2 "Package_SO:SOIC-16W_7.5x10.3mm_P1.27mm" H 3200 3050 50  0001 C CNN
-F 3 "http://datasheets.maximintegrated.com/en/ds/DS3231.pdf" H 3470 3700 50  0001 C CNN
-	1    3200 3650
-	1    0    0    -1
-$EndComp
-$Comp
 L Chicken~Coop~Door:Buck_Boost_module U6
 U 1 1 5CEF5879
@@
 Connection ~ 7200 2550
 Wire Wire Line
-	7200 2550 7200 3300
+	7200 2550 7200 2700
 Wire Wire Line
 	5650 2450 7300 2450
 Connection ~ 7300 2450
 Wire Wire Line
-	7300 2450 7300 3400
+	7300 2450 7300 2800
 Wire Wire Line
 	2250 4750 2350 4750
@@
 F 0 "R4" V 3150 2250 50  0000 L CNN
 F 1 "1k" V 3320 2255 50  0000 L CNN
-F 2 "" V 3180 2300 50  0001 C CNN
+F 2 "Resistor_THT:R_Axial_DIN0204_L3.6mm_D1.6mm_P7.62mm_Horizontal" V 3180 2300 50  0001 C CNN
 F 3 "~" H 3250 2300 50  0001 C CNN
 	1    3250 2300
@@
 $EndComp
 Wire Wire Line
-	4150 1800 5550 1800
-Wire Wire Line
-	4150 1650 5650 1650
-$Comp
-L power:GND #PWR?
+	4150 1800 5300 1800
+Wire Wire Line
+	4150 1650 5200 1650
+$Comp
+L power:GND #PWR0115
 U 1 1 5CF9556B
 P 3750 2500
-F 0 "#PWR?" H 3750 2250 50  0001 C CNN
+F 0 "#PWR0115" H 3750 2250 50  0001 C CNN
 F 1 "GND" H 3755 2327 50  0000 C CNN
 F 2 "" H 3750 2500 50  0001 C CNN
@@
 D10
 Wire Wire Line
-	3700 3750 4900 3750
-Wire Wire Line
 	3750 2100 3750 1950
-Wire Wire Line
-	2250 1800 2250 4750
-Wire Wire Line
-	1950 1650 1950 4950
 Wire Wire Line
 	5550 1800 5550 2550
@@
 	8050 3400 8250 3400
 Connection ~ 8250 3400
+$Comp
+L sensors:SSD1306_OLED_128x32 U4
+U 1 1 5EBCC666
+P 6150 5850
+F 0 "U4" H 6778 5951 50  0000 L CNN
+F 1 "SSD1306_OLED_128x32" H 6778 5860 50  0000 L CNN
+F 2 "personal:SSD1306_Adafruit_128x32" H 5650 6200 50  0001 C CNN
+F 3 "" H 5650 6200 50  0001 C CNN
+	1    6150 5850
+	1    0    0    -1
+$EndComp
+Wire Wire Line
+	5400 4750 5400 5650
+Wire Wire Line
+	5550 5650 5400 5650
+Wire Wire Line
+	5550 5750 5500 5750
+Wire Wire Line
+	5500 4750 5500 5750
+Wire Wire Line
+	5250 5850 5550 5850
+Wire Wire Line
+	5250 5950 5550 5950
+$Comp
+L sensors:DS3231 U2
+U 1 1 5EC037F4
+P 3350 3350
+F 0 "U2" H 3350 3765 50  0000 C CNN
+F 1 "DS3231" H 3350 3674 50  0000 C CNN
+F 2 "Connector_PinSocket_2.54mm:PinSocket_1x06_P2.54mm_Vertical" H 3700 3000 50  0001 C CNN
+F 3 "" H 3700 3000 50  0001 C CNN
+	1    3350 3350
+	1    0    0    -1
+$EndComp
+Wire Wire Line
+	3000 3300 2700 3300
+Wire Wire Line
+	2700 3300 2700 3750
+$Comp
+L Connector_Generic:Conn_01x01 J8
+U 1 1 5EC15455
+P 4300 2250
+F 0 "J8" V 4173 2330 50  0000 L CNN
+F 1 "Conn_01x01" V 4264 2330 50  0000 L CNN
+F 2 "TestPoint:TestPoint_THTPad_D2.0mm_Drill1.0mm" H 4300 2250 50  0001 C CNN
+F 3 "~" H 4300 2250 50  0001 C CNN
+	1    4300 2250
+	0    1    1    0
+$EndComp
+Wire Wire Line
+	2700 3750 4900 3750
+$Comp
+L Connector_Generic:Conn_01x02 J9
+U 1 1 5EC2617A
+P 1600 3700
+F 0 "J9" H 1680 3692 50  0000 L CNN
+F 1 "BuckBoost" H 1680 3601 50  0000 L CNN
+F 2 "Connector_JST:JST_XH_B02B-XH-A_1x02_P2.50mm_Vertical" H 1600 3700 50  0001 C CNN
+F 3 "~" H 1600 3700 50  0001 C CNN
+	1    1600 3700
+	-1   0    0    -1
+$EndComp
+$Comp
+L Connector_Generic:Conn_01x02 J10
+U 1 1 5EC4F65E
+P 5000 1400
+F 0 "J10" H 5080 1392 50  0000 L CNN
+F 1 "Charger" H 5080 1301 50  0000 L CNN
+F 2 "Connector_JST:JST_XH_B02B-XH-A_1x02_P2.50mm_Vertical" H 5000 1400 50  0001 C CNN
+F 3 "~" H 5000 1400 50  0001 C CNN
+	1    5000 1400
+	-1   0    0    -1
+$EndComp
+Wire Wire Line
+	2250 1800 2250 3700
+Wire Wire Line
+	1950 1650 1950 3800
+Wire Wire Line
+	1800 3700 2250 3700
+Connection ~ 2250 3700
+Wire Wire Line
+	2250 3700 2250 4750
+Wire Wire Line
+	1800 3800 1950 3800
+Connection ~ 1950 3800
+Wire Wire Line
+	1950 3800 1950 4950
+Wire Wire Line
+	5200 1500 5200 1650
+Connection ~ 5200 1650
+Wire Wire Line
+	5200 1650 5650 1650
+Wire Wire Line
+	5200 1400 5300 1400
+Wire Wire Line
+	5300 1400 5300 1800
+Connection ~ 5300 1800
+Wire Wire Line
+	5300 1800 5550 1800
+$Comp
+L Connector_Generic:Conn_01x02 J11
+U 1 1 5EC5D176
+P 7700 2700
+F 0 "J11" H 7780 2692 50  0000 L CNN
+F 1 "Charger" H 7780 2601 50  0000 L CNN
+F 2 "Connector_JST:JST_XH_B02B-XH-A_1x02_P2.50mm_Vertical" H 7700 2700 50  0001 C CNN
+F 3 "~" H 7700 2700 50  0001 C CNN
+	1    7700 2700
+	1    0    0    -1
+$EndComp
+Wire Wire Line
+	7500 2700 7200 2700
+Connection ~ 7200 2700
+Wire Wire Line
+	7200 2700 7200 3300
+Wire Wire Line
+	7300 2800 7500 2800
+Connection ~ 7300 2800
+Wire Wire Line
+	7300 2800 7300 3400
+Wire Wire Line
+	3750 1950 4300 1950
+Connection ~ 3750 1950
+Wire Wire Line
+	4300 1950 4300 2050
 $EndSCHEMATC

Commit message: PCB layout complete
Parts:
- J1: footprint (none) -> Connector_PinHeader_2.54mm:PinHeader_1x06_P2.54mm_Vertical
Changed lines of the file:
@@
 F 0 "J1" V 5712 2844 50  0000 L CNN
 F 1 "Programming_Headers" V 5803 2844 50  0000 L CNN
-F 2 "" H 5650 2600 50  0001 C CNN
+F 2 "Connector_PinHeader_2.54mm:PinHeader_1x06_P2.54mm_Vertical" H 5650 2600 50  0001 C CNN
 F 3 "~" H 5650 2600 50  0001 C CNN
 	1    5650 2600
@@
 Wire Wire Line
 	5550 3050 5550 2800
-Wire Wire Line
-	5650 2800 5650 3050
 Wire Wire Line
 	5750 3050 5750 2800
@@
 Wire Wire Line
 	4300 1950 4300 2050
+Wire Wire Line
+	5650 2800 5650 3050
 $EndSCHEMATC
